Commit message: til that base

File: urdf/med7.xacro (robot description, xacro)
@@ -9,4 +9,5 @@
     <xacro:arg name="tool" default="sca"/>
     <xacro:arg name="parent_link" default="lbr_link_ee"/>
+    <xacro:arg name="tilt_angle" default="-0.5" /> <!-- Tilt angle in radians (about -29 degrees forward) -->
     <!-- KDL requires a link without inertia / Gazebo requires a connection to world link or robot
     will tipple https://github.com/lbr-stack/lbr_fri_ros2_stack/issues/230 -->
@@ -17,4 +18,5 @@
         <parent link="world" />
         <child link="$(arg robot_name)_link_0" />
+        <origin rpy="$(arg tilt_angle) 0 0" xyz="0 0 0" />
     </joint>
     <!-- med -->

Commit message: Enhance integration with new launch files for hardware and mock robots, update RCM management to utilize TF for pose tracking, and improve GUI and teleoperation controls for smoother operation. Refactor pose handling in the GUI and IK solver for better performance and compatibility.

File: urdf/med7.xacro (robot description, xacro)
@@ -9,5 +9,5 @@
     <xacro:arg name="tool" default="sca"/>
     <xacro:arg name="parent_link" default="lbr_link_ee"/>
-    <xacro:arg name="tilt_angle" default="-1.0" /> <!-- Tilt angle in radians (about -57 degrees forward) -->
+    <xacro:arg name="tilt_angle" default="0.0" /> <!-- No tilt - robot stands upright -->
     <!-- KDL requires a link without inertia / Gazebo requires a connection to world link or robot
     will tipple https://github.com/lbr-stack/lbr_fri_ros2_stack/issues/230 -->

File: urdf/psm.classic.urdf.xacro (robot description, xacro)
@@ -41,5 +41,5 @@
         <parent link="${parent_link}"/>
         <child link="base_link"/>
-        <origin xyz="0 0 0.02" rpy="${PI/2} 0 0"/>
+        <origin xyz="0 0 0.02" rpy="${PI/2} 0 ${PI/2}"/>
     </joint>
     <!-- Joint 2: Connect adaptor base_link to PSM base -->
