Commit message: hardware speed adjustment

File: urdf/psm.classic.urdf.xacro (robot description, xacro)
@@ -41,5 +41,5 @@
         <parent link="${parent_link}"/>
         <child link="base_link"/>
-        <origin xyz="0 0 0.02" rpy="${PI/2} 0 ${PI/2}"/>
+        <origin xyz="0 0 0.02" rpy="${PI/2} 0 ${-PI/2}"/>
     </joint>
     <!-- Joint 2: Connect adaptor base_link to PSM base -->
